File: hardware/Pomodoro_timer/Pomodoro_timer.kicad_sch (KiCad schematic)
At the start: 0 parts

Commit message: PCB Ver.A All changes finalized & PCB design has been started
Other:
- added sheet MCU_Misc (MCU_Misc.kicad_sch)
Changed lines of the file:
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@@
+	)
+	(sheet
+		(at 16.51 73.66)
+		(size 189.23 64.77)
+		(exclude_from_sim no)
+		(in_bom yes)
+		(on_board yes)
+		(dnp no)
+		(fields_autoplaced yes)
+		(stroke
+			(width 0.1524)
+			(type solid)
+		)
+		(fill
+			(color 0 0 0 0.0000)
+		)
+		(property "Sheetname" "MCU_Misc"
+			(at 16.51 72.9484 0)
+			(effects
+				(font
+					(size 1.27 1.27)
+				)
+				(justify left bottom)
+			)
+		)
+		(property "Sheetfile" "MCU_Misc.kicad_sch"
+			(at 16.51 139.0146 0)
+			(effects
+				(font
+					(size 1.27 1.27)
+				)
+				(justify left top)
+			)
+		)
+		(instances
+			(project "Pomodoro_timer"
+				(path "/de804b87-618c-4b40-9e9d-dfdac3d4076a"
+					(page "4")
+				)
+			)
+		)
 	)
 	(sheet
