File: hardware/Pomodoro_timer/TM1637_Display.kicad_sch (KiCad schematic)
At the start: 0 parts

Commit message: TM1637 Design started
Parts:
- added C5: 100nF, symbol Device:C_Small
- added U4: CC56-12EWA, Display_7Segment:CA56-12EWA, symbol Display_Character:CC56-12EWA
- added U5: TM1637, TM1637:DIP778W43P254L2612H431Q20N, symbol TM1637:TM1637
Connections:
- new net: U4.1 (e), U5.6 (SEG5/KS5)
- new net: U4.10 (f), U5.7 (SEG6/KS6)
- new net: U4.11 (a), U5.2 (SEG1/KS1)
- new net: U4.12 (CC1), U5.15 (GRID1)
- new net: U4.2 (d), U5.5 (SEG4/KS4)
- new net: U4.3 (DPX), U5.9 (SEG8/KS8)
- new net: U4.4 (c), U5.4 (SEG3/KS3)
- new net: U4.5 (g), U5.8 (SEG7/KS7)
- new net: U4.6 (CC4), U5.12 (GRID4)
- new net: U4.7 (b), U5.3 (SEG2/KS2)
- new net: U4.8 (CC3), U5.13 (GRID3)
- new net: U4.9 (CC2), U5.14 (GRID2)
- new net GND: C5.2, U5.1 (GND)
- new net PWR: C5.1, U5.16 (VDD)
- no-connect marks 0 -> 4

Commit message: PCB Ver.A All changes finalized & PCB design has been started
Parts:
- added R8, R9: 4K7, Resistor_SMD:R_1206_3216Metric_Pad1.30x1.75mm_HandSolder, symbol Device:R_Small
- C5: footprint (none) -> Capacitor_SMD:C_1206_3216Metric_Pad1.33x1.80mm_HandSolder
- U4: renamed from U5; footprint TM1637:DIP778W43P254L2612H431Q20N -> Package_SO:SOIC-20W_7.5x12.8mm_P1.27mm
- renumbered U4 to U5
Connections:
- net PWR: now also R8.1, R9.1
- net DIO: now reaches U4.17 (DIO)
- net DIO: now also R8.2
- net CLK: now reaches U4.18 (CLK)
- net CLK: now also R9.2
